Commit message: feat: add simulated GPS (NavSat) sensor
- Add gps_link/gps_joint to URDF, mounted on top of trunk
- Add Gazebo NavSat sensor plugin with standard u-blox noise (0.5 m
  horizontal, 0.8 m vertical std dev)
- Add gz-sim-navsat-system plugin to world SDF (required for sensor activation)
- Add spherical_coordinates to world SDF to produce real lat/lon output
- Bridge /gps/fix (gz.msgs.NavSat -> sensor_msgs/msg/NavSatFix) in launch file
- Update README: mark GPS as implemented, add usage and configuration notes

File: unitree_go2_description/urdf/unitree_go2_gazebo.xacro (robot description, xacro)
@@ -93,4 +93,43 @@
                     <initial_orientation_as_reference>false</initial_orientation_as_reference>
                 </plugin>
+            </sensor>
+        </gazebo>
+        <!-- GPS / NavSat plugin — simulates u-blox standard GPS (~0.5 m horizontal noise) -->
+        <gazebo reference="gps_link">
+            <sensor name="navsat_sensor" type="navsat">
+                <always_on>true</always_on>
+                <update_rate>10</update_rate>
+                <topic>gps/fix</topic>
+                <gz_frame_id>gps_link</gz_frame_id>
+                <navsat>
+                    <position_sensing>
+                        <horizontal>
+                            <noise type="gaussian">
+                                <mean>0.0</mean>
+                                <stddev>0.5</stddev>
+                            </noise>
+                        </horizontal>
+                        <vertical>
+                            <noise type="gaussian">
+                                <mean>0.0</mean>
+                                <stddev>0.8</stddev>
+                            </noise>
+                        </vertical>
+                    </position_sensing>
+                    <velocity_sensing>
+                        <horizontal>
+                            <noise type="gaussian">
+                                <mean>0.0</mean>
+                                <stddev>0.1</stddev>
+                            </noise>
+                        </horizontal>
+                        <vertical>
+                            <noise type="gaussian">
+                                <mean>0.0</mean>
+                                <stddev>0.1</stddev>
+                            </noise>
+                        </vertical>
+                    </velocity_sensing>
+                </navsat>
             </sensor>
         </gazebo>

File: unitree_go2_description/urdf/unitree_go2_robot.xacro (robot description, xacro)
@@ -66,4 +66,32 @@
         <origin rpy="0 0 0" xyz="0 0 0" />
     </joint>
+    <!-- GPS link — mounted on top center of trunk -->
+    <joint name="gps_joint" type="fixed">
+        <parent link="trunk" />
+        <child link="gps_link" />
+        <origin rpy="0 0 0" xyz="0.0 0.0 0.065" />
+    </joint>
+    <link name="gps_link">
+        <inertial>
+            <mass value="0.001" />
+            <origin rpy="0 0 0" xyz="0 0 0" />
+            <inertia ixx="0.0001" ixy="0" ixz="0" iyy="0.0001" iyz="0" izz="0.0001" />
+        </inertial>
+        <visual>
+            <origin rpy="0 0 0" xyz="0 0 0" />
+            <geometry>
+                <box size="0.05 0.05 0.02" />
+            </geometry>
+            <material name="white">
+                <color rgba="1 1 1 1" />
+            </material>
+        </visual>
+        <collision>
+            <origin rpy="0 0 0" xyz="0 0 0" />
+            <geometry>
+                <box size="0.05 0.05 0.02" />
+            </geometry>
+        </collision>
+    </link>
     <link name="imu_link">
         <inertial>
